Commit message: ROS 2 Control Hardware basic hardware interface

File: so_arm_config/config/so_arm_101.ros2_control.xacro (robot description, xacro)
@@ -1,10 +1,16 @@
 <?xml version="1.0"?>
 <robot xmlns:xacro="http://www.ros.org/wiki/xacro">
-    <xacro:macro name="so_arm_101_ros2_control" params="name initial_positions_file">
+    <xacro:macro name="so_arm_101_ros2_control" params="name initial_positions_file mock:=false">
         <xacro:property name="initial_positions" value="${load_yaml(initial_positions_file)['initial_positions']}"/>
         <ros2_control name="${name}" type="system">
             <hardware>
-                <!-- By default, set up controllers for simulation. This won't work on real hardware -->
-                <plugin>mock_components/GenericSystem</plugin>
+                <!-- Set up controllers for simulation. This won't work on real hardware -->
+                <xacro:if value="${mock}">
+                  <plugin>mock_components/GenericSystem</plugin>
+                </xacro:if>
+                <xacro:unless value="${mock}">
+                  <plugin>so_arm_controllers/SOArmHardwareInterface</plugin>
+                </xacro:unless>
+                <!-- Set up controllers for real info send. Can work with real robot or virtual controller. -->
             </hardware>
             <joint name="shoulder_pan">

Commit message: Moveit configuration correction

File: so_arm_config/config/so_arm_101.ros2_control.xacro (robot description, xacro)
@@ -1,5 +1,5 @@
 <?xml version="1.0"?>
 <robot xmlns:xacro="http://www.ros.org/wiki/xacro">
-    <xacro:macro name="so_arm_101_ros2_control" params="name initial_positions_file mock:=false">
+    <xacro:macro name="so_arm_101_ros2_control" params="name initial_positions_file mock:=true">
         <xacro:property name="initial_positions" value="${load_yaml(initial_positions_file)['initial_positions']}"/>
         <ros2_control name="${name}" type="system">
@@ -17,60 +17,48 @@
                 <command_interface name="position"/>
                 <command_interface name="velocity"/>
-                <command_interface name="effort"/>
                 <state_interface name="position">
                   <param name="initial_value">${initial_positions['shoulder_pan']}</param>
                 </state_interface>
                 <state_interface name="velocity"/>
-                <state_interface name="effort"/>
             </joint>
             <joint name="shoulder_lift">
                 <command_interface name="position"/>
                 <command_interface name="velocity"/>
-                <command_interface name="effort"/>
                 <state_interface name="position">
                   <param name="initial_value">${initial_positions['shoulder_lift']}</param>
                 </state_interface>
                 <state_interface name="velocity"/>
-                <state_interface name="effort"/>
             </joint>
             <joint name="elbow_flex">
                 <command_interface name="position"/>
                 <command_interface name="velocity"/>
-                <command_interface name="effort"/>
                 <state_interface name="position">
                   <param name="initial_value">${initial_positions['elbow_flex']}</param>
                 </state_interface>
                 <state_interface name="velocity"/>
-                <state_interface name="effort"/>
             </joint>
             <joint name="wrist_flex">
                 <command_interface name="position"/>
                 <command_interface name="velocity"/>
-                <command_interface name="effort"/>
                 <state_interface name="position">
                   <param name="initial_value">${initial_positions['wrist_flex']}</param>
                 </state_interface>
                 <state_interface name="velocity"/>
-                <state_interface name="effort"/>
             </joint>
             <joint name="wrist_roll">
                 <command_interface name="position"/>
                 <command_interface name="velocity"/>
-                <command_interface name="effort"/>
                 <state_interface name="position">
                   <param name="initial_value">${initial_positions['wrist_roll']}</param>
                 </state_interface>
                 <state_interface name="velocity"/>
-                <state_interface name="effort"/>
             </joint>
             <joint name="gripper">
                 <command_interface name="position"/>
                 <command_interface name="velocity"/>
-                <command_interface name="effort"/>
                 <state_interface name="position">
                   <param name="initial_value">${initial_positions['gripper']}</param>
                 </state_interface>
                 <state_interface name="velocity"/>
-                <state_interface name="effort"/>
             </joint>
         </ros2_control>

File: so_arm_config/config/so_arm_101.urdf.xacro (robot description, xacro)
@@ -6,4 +6,4 @@
     <!-- Import control_xacro -->
     <xacro:include filename="so_arm_101.ros2_control.xacro" />
-    <xacro:so_arm_101_ros2_control name="FakeSystem" initial_positions_file="$(arg initial_positions_file)"/>
+    <xacro:so_arm_101_ros2_control name="SO-ARM101" initial_positions_file="$(arg initial_positions_file)"/>
 </robot>

Commit message: Adding option to switch between simulation and real controller

File: so_arm_config/config/so_arm_101.ros2_control.xacro (robot description, xacro)
@@ -1,16 +1,20 @@
 <?xml version="1.0"?>
 <robot xmlns:xacro="http://www.ros.org/wiki/xacro">
-    <xacro:macro name="so_arm_101_ros2_control" params="name initial_positions_file mock:=true">
-        <xacro:property name="initial_positions" value="${load_yaml(initial_positions_file)['initial_positions']}"/>
+    <xacro:macro name="so_arm_101_ros2_control"
+      params="name initial_positions_file mock_controller:=true">
+        <xacro:property
+          name="initial_positions"
+          value="${xacro.load_yaml(initial_positions_file)['initial_positions']}"
+        />
         <ros2_control name="${name}" type="system">
             <hardware>
-                <!-- Set up controllers for simulation. This won't work on real hardware -->
-                <xacro:if value="${mock}">
+                <!-- Set up controllers for mock_controller. This won't work on real hardware -->
+                <xacro:if value="${mock_controller}">
                   <plugin>mock_components/GenericSystem</plugin>
                 </xacro:if>
-                <xacro:unless value="${mock}">
+                <!-- Set up controllers for real info send. Can work with real robot or virtual controller. -->
+                <xacro:unless value="${mock_controller}">
                   <plugin>so_arm_controllers/SOArmHardwareInterface</plugin>
                 </xacro:unless>
-                <!-- Set up controllers for real info send. Can work with real robot or virtual controller. -->
             </hardware>
             <joint name="shoulder_pan">

File: so_arm_config/config/so_arm_101.urdf.xacro (robot description, xacro)
@@ -2,8 +2,12 @@
 <robot xmlns:xacro="http://www.ros.org/wiki/xacro" name="so_arm_101">
     <xacro:arg name="initial_positions_file" default="initial_positions.yaml" />
+    <xacro:arg name="mock_controller" default="false" />
     <!-- Import so_arm_101 urdf file -->
     <xacro:include filename="$(find so_arm_description)/urdf/so_arm_101.urdf.xacro" />
     <!-- Import control_xacro -->
     <xacro:include filename="so_arm_101.ros2_control.xacro" />
-    <xacro:so_arm_101_ros2_control name="SO-ARM101" initial_positions_file="$(arg initial_positions_file)"/>
+    <xacro:so_arm_101_ros2_control name="SO-ARM101"
+        initial_positions_file="$(arg initial_positions_file)"
+        mock_controller="$(arg mock_controller)"
+    />
 </robot>
