Commit message: Launch for robot visualization

File: so_arm_description/urdf/so_arm_101.urdf.xacro (robot description, xacro)
@@ -5,4 +5,5 @@
     <color rgba="0.8 0.8 0.8 1.0"/>
   </material>
+  <!-- TODO: Uncomment the material tags when multiple visual materials are working on RVIZ -->
   <material name="sts3215">
     <color rgba="0.1 0.1 0.1 1.0"/>
@@ -52,5 +53,5 @@
         <mesh filename="package://so_arm_description/meshes/sts3215_03a_v1.stl"/>
       </geometry>
-      <material name="sts3215"/>
+      <!-- <material name="sts3215"/> -->
     </visual>
     <collision>
@@ -91,5 +92,6 @@
         <mesh filename="package://so_arm_description/meshes/sts3215_03a_v1.stl"/>
       </geometry>
-      <material name="sts3215"/>
+      <!-- <material name="sts3215"/> -->
+      <material name="3d_printed"/>
     </visual>
     <collision>
@@ -144,5 +146,6 @@
         <mesh filename="package://so_arm_description/meshes/sts3215_03a_v1.stl"/>
       </geometry>
-      <material name="sts3215"/>
+      <material name="3d_printed"/>
+      <!-- <material name="sts3215"/> -->
     </visual>
     <collision>
@@ -211,5 +214,5 @@
         <mesh filename="package://so_arm_description/meshes/sts3215_03a_v1.stl"/>
       </geometry>
-      <material name="sts3215"/>
+      <!-- <material name="sts3215"/> -->
     </visual>
     <collision>
@@ -236,5 +239,6 @@
         <mesh filename="package://so_arm_description/meshes/sts3215_03a_no_horn_v1.stl"/>
       </geometry>
-      <material name="sts3215"/>
+      <material name="3d_printed"/>
+      <!-- <material name="sts3215"/> -->
     </visual>
     <collision>
@@ -275,5 +279,6 @@
         <mesh filename="package://so_arm_description/meshes/sts3215_03a_v1.stl"/>
       </geometry>
-      <material name="sts3215"/>
+      <material name="3d_printed"/>
+      <!-- <material name="sts3215"/> -->
     </visual>
     <collision>

Commit message: Reordening joints from base to tip

File: so_arm_description/urdf/so_arm_101.urdf.xacro (robot description, xacro)
@@ -76,4 +76,22 @@
     </collision>
   </link>
+  <!-- Joint from base to shoulder -->
+  <joint name="shoulder_pan" type="revolute">
+    <origin xyz="0.0388353 0 0.0624" rpy="${pi} 0 ${-pi}"/>
+    <parent link="base_link"/>
+    <child link="shoulder_link"/>
+    <axis xyz="0 0 1"/>
+    <limit effort="10" velocity="10" lower="-1.91986" upper="1.91986"/>
+  </joint>
+  <transmission name="shoulder_pan_trans">
+    <type>transmission_interface/SimpleTransmission</type>
+    <joint name="shoulder_pan">
+      <hardwareInterface>hardware_interface/PositionJointInterface</hardwareInterface>
+    </joint>
+    <actuator name="motor1">
+      <hardwareInterface>hardware_interface/PositionJointInterface</hardwareInterface>
+      <mechanicalReduction>1</mechanicalReduction>
+    </actuator>
+  </transmission>
   <!-- Link shoulder -->
   <link name="shoulder_link">
@@ -130,4 +148,22 @@
     </collision>
   </link>
+  <!-- Joint from shoulder to upper_arm -->
+  <joint name="shoulder_lift" type="revolute">
+    <origin xyz="-0.0303992 -0.0182778 -0.0542" rpy="${-pi/2} ${-pi/2} 0"/>
+    <parent link="shoulder_link"/>
+    <child link="upper_arm_link"/>
+    <axis xyz="0 0 1"/>
+    <limit effort="10" velocity="10" lower="-1.74533" upper="1.74533"/>
+  </joint>
+  <transmission name="shoulder_lift_trans">
+    <type>transmission_interface/SimpleTransmission</type>
+    <joint name="shoulder_lift">
+      <hardwareInterface>hardware_interface/PositionJointInterface</hardwareInterface>
+    </joint>
+    <actuator name="motor2">
+      <hardwareInterface>hardware_interface/PositionJointInterface</hardwareInterface>
+      <mechanicalReduction>1</mechanicalReduction>
+    </actuator>
+  </transmission>
   <!-- Link upper_arm -->
   <link name="upper_arm_link">
@@ -170,231 +206,4 @@
     </collision>
   </link>
-  <!-- Link lower_arm -->
-  <link name="lower_arm_link">
-    <inertial>
-      <origin xyz="-0.0980701 0.00324376 0.0182831" rpy="0 0 0"/>
-      <mass value="0.104"/>
-      <inertia
-        ixx="2.87438e-05" ixy="7.41152e-06" ixz="1.26409e-06"
-        iyy="0.000159844" iyz="-4.90188e-08" izz="0.00014529"
-      />
-    </inertial>
-    <!-- Part under_arm_so101_v1 -->
-    <visual>
-      <origin xyz="-0.0648499 -0.032 0.0182" rpy="${pi} 0 0"/>
-      <geometry>
-        <mesh filename="package://so_arm_description/meshes/under_arm_so101_v1.stl"/>
-      </geometry>
-      <material name="3d_printed"/>
-    </visual>
-    <collision>
-      <origin xyz="-0.0648499 -0.032 0.0182" rpy="${pi} 0 0"/>
-      <geometry>
-        <mesh filename="package://so_arm_description/meshes/under_arm_so101_v1.stl"/>
-      </geometry>
-    </collision>
-    <!-- Part motor_holder_so101_wrist_v1 -->
-    <visual>
-      <origin xyz="-0.0648499 -0.032 0.018" rpy="${-pi} 0 0"/>
-      <geometry>
-        <mesh filename="package://so_arm_description/meshes/motor_holder_so101_wrist_v1.stl"/>
-      </geometry>
-      <material name="3d_printed"/>
-    </visual>
-    <collision>
-      <origin xyz="-0.0648499 -0.032 0.018" rpy="${-pi} 0 0"/>
-      <geometry>
-        <mesh filename="package://so_arm_description/meshes/motor_holder_so101_wrist_v1.stl"/>
-      </geometry>
-    </collision>
-    <!-- Part sts3215_03a_v1_4 -->
-    <visual>
-      <origin xyz="-0.1224 0.0052 0.0187" rpy="${-pi} 0 ${-pi}"/>
-      <geometry>
-        <mesh filename="package://so_arm_description/meshes/sts3215_03a_v1.stl"/>
-      </geometry>
-      <!-- <material name="sts3215"/> -->
-    </visual>
-    <collision>
-      <origin xyz="-0.1224 0.0052 0.0187" rpy="${-pi} 0 ${-pi}"/>
-      <geometry>
-        <mesh filename="package://so_arm_description/meshes/sts3215_03a_v1.stl"/>
-      </geometry>
-    </collision>
-  </link>
-  <!-- Link wrist -->
-  <link name="wrist_link">
-    <inertial>
-      <origin xyz="-0.000103312 -0.0386143 0.0281156" rpy="0 0 0"/>
-      <mass value="0.079"/>
-      <inertia
-        ixx="3.68263e-05" ixy="1.7893e-08" ixz="-5.28128e-08"
-        iyy="2.5391e-05" iyz="3.6412e-06" izz="2.1e-05"
-      />
-    </inertial>
-    <!-- Part sts3215_03a_no_horn_v1 -->
-    <visual>
-      <origin xyz="0 -0.0424 0.0306" rpy="${pi/2} ${pi/2} 0"/>
-      <geometry>
-        <mesh filename="package://so_arm_description/meshes/sts3215_03a_no_horn_v1.stl"/>
-      </geometry>
-      <material name="3d_printed"/>
-      <!-- <material name="sts3215"/> -->
-    </visual>
-    <collision>
-      <origin xyz="0 -0.0424 0.0306" rpy="${pi/2} ${pi/2} 0"/>
-      <geometry>
-        <mesh filename="package://so_arm_description/meshes/sts3215_03a_no_horn_v1.stl"/>
-      </geometry>
-    </collision>
-    <!-- Part wrist_roll_pitch_so101_v2 -->
-    <visual>
-      <origin xyz="0 -0.028 0.0181" rpy="${-pi/2} ${-pi/2} 0"/>
-      <geometry>
-        <mesh filename="package://so_arm_description/meshes/wrist_roll_pitch_so101_v2.stl"/>
-      </geometry>
-      <material name="3d_printed"/>
-    </visual>
-    <collision>
-      <origin xyz="0 -0.028 0.0181" rpy="${-pi/2} ${-pi/2} 0"/>
-      <geometry>
-        <mesh filename="package://so_arm_description/meshes/wrist_roll_pitch_so101_v2.stl"/>
-      </geometry>
-    </collision>
-  </link>
-  <!-- Link gripper -->
-  <link name="gripper_link">
-    <inertial>
-      <origin xyz="0.000213627 0.000245138 -0.025187" rpy="0 0 0"/>
-      <mass value="0.087"/>
-      <inertia
-        ixx="2.75087e-05" ixy="-3.35241e-07" ixz="-5.7352e-06"
-        iyy="4.33657e-05" iyz="-5.17847e-08" izz="3.45059e-05"
-      />
-    </inertial>
-    <!-- Part sts3215_03a_v1_5 -->
-    <visual>
-      <origin xyz="0.0077 0.0001 -0.0234" rpy="${-pi/2} 0 0"/>
-      <geometry>
-        <mesh filename="package://so_arm_description/meshes/sts3215_03a_v1.stl"/>
-      </geometry>
-      <material name="3d_printed"/>
-      <!-- <material name="sts3215"/> -->
-    </visual>
-    <collision>
-      <origin xyz="0.0077 0.0001 -0.0234" rpy="${-pi/2} 0 0"/>
-      <geometry>
-        <mesh filename="package://so_arm_description/meshes/sts3215_03a_v1.stl"/>
-      </geometry>
-    </collision>
-    <!-- Part wrist_roll_follower_so101_v1 -->
-    <visual>
-      <origin xyz="0 -0.000218214 0.000949706" rpy="${-pi} 0 0"/>
-      <geometry>
-        <mesh filename="package://so_arm_description/meshes/wrist_roll_follower_so101_v1.stl"/>
-      </geometry>
-      <material name="3d_printed"/>
-    </visual>
-    <collision>
-      <origin xyz="0 -0.000218214 0.000949706" rpy="${-pi} 0 0"/>
-      <geometry>
-        <mesh filename="package://so_arm_description/meshes/wrist_roll_follower_so101_v1.stl"/>
-      </geometry>
-    </collision>
-  </link>
-  <!-- Gripper frame (dummy link + fixed joint) -->
-  <link name="gripper_frame_link">
-    <origin xyz="0 0 0" rpy="0 -0 0"/>
-    <inertial>
-      <origin xyz="0 0 0" rpy="0 0 0"/>
-      <mass value="1e-9"/>
-      <inertia ixx="0" ixy="0" ixz="0" iyy="0" iyz="0" izz="0"/>
-    </inertial>
-  </link>
-  <joint name="gripper_frame_joint" type="fixed">
-    <origin xyz="-0.0079 -0.000218121 -0.0981274" rpy="0 ${pi} 0"/>
-    <parent link="gripper_link"/>
-    <child link="gripper_frame_link"/>
-    <axis xyz="0 0 0"/>
-  </joint>
-  <!-- Link moving_jaw_so101_v1 -->
-  <link name="moving_jaw_so101_v1_link">
-    <inertial>
-      <origin xyz="-0.00157495 -0.0300244 0.0192755" rpy="0 0 0"/>
-      <mass value="0.012"/>
-      <inertia
-        ixx="6.61427e-06" ixy="-3.19807e-07" ixz="-5.90717e-09"
-        iyy="1.89032e-06" iyz="-1.09945e-07" izz="5.28738e-06"
-      />
-    </inertial>
-    <!-- Part moving_jaw_so101_v1 -->
-    <visual>
-      <origin xyz="0 0 0.0189" rpy="0 0 0"/>
-      <geometry>
-        <mesh filename="package://so_arm_description/meshes/moving_jaw_so101_v1.stl"/>
-      </geometry>
-      <material name="3d_printed"/>
-    </visual>
-    <collision>
-      <origin xyz="0 0 0.0189" rpy="0 0 0"/>
-      <geometry>
-        <mesh filename="package://so_arm_description/meshes/moving_jaw_so101_v1.stl"/>
-      </geometry>
-    </collision>
-  </link>
-  <!-- Joint from gripper to moving_jaw_so101_v1 -->
-  <joint name="gripper" type="revolute">
-    <origin xyz="0.0202 0.0188 -0.0234" rpy="${pi/2} 0 0"/>
-    <parent link="gripper_link"/>
-    <child link="moving_jaw_so101_v1_link"/>
-    <axis xyz="0 0 1"/>
-    <limit effort="10" velocity="10" lower="-0.174533" upper="1.74533"/>
-  </joint>
-  <transmission name="gripper_trans">
-    <type>transmission_interface/SimpleTransmission</type>
-    <joint name="gripper">
-      <hardwareInterface>hardware_interface/PositionJointInterface</hardwareInterface>
-    </joint>
-    <actuator name="motor6">
-      <hardwareInterface>hardware_interface/PositionJointInterface</hardwareInterface>
-      <mechanicalReduction>1</mechanicalReduction>
-    </actuator>
-  </transmission>
-  <!-- Joint from wrist to gripper -->
-  <joint name="wrist_roll" type="revolute">
-    <origin xyz="0 -0.0611 0.0181" rpy="${pi/2} 0.0486795 ${pi}"/>
-    <parent link="wrist_link"/>
-    <child link="gripper_link"/>
-    <axis xyz="0 0 1"/>
-    <limit effort="10" velocity="10" lower="-2.74385" upper="2.84121"/>
-  </joint>
-  <transmission name="wrist_roll_trans">
-    <type>transmission_interface/SimpleTransmission</type>
-    <joint name="wrist_roll">
-      <hardwareInterface>hardware_interface/PositionJointInterface</hardwareInterface>
-    </joint>
-    <actuator name="motor5">
-      <hardwareInterface>hardware_interface/PositionJointInterface</hardwareInterface>
-      <mechanicalReduction>1</mechanicalReduction>
-    </actuator>
-  </transmission>
-  <!-- Joint from lower_arm to wrist -->
-  <joint name="wrist_flex" type="revolute">
-    <origin xyz="-0.1349 0.0052 0" rpy="0 0 ${-pi/2}"/>
-    <parent link="lower_arm_link"/>
-    <child link="wrist_link"/>
-    <axis xyz="0 0 1"/>
-    <limit effort="10" velocity="10" lower="-1.65806" upper="1.65806"/>
-  </joint>
-  <transmission name="wrist_flex_trans">
-    <type>transmission_interface/SimpleTransmission</type>
-    <joint name="wrist_flex">
-      <hardwareInterface>hardware_interface/PositionJointInterface</hardwareInterface>
-    </joint>
-    <actuator name="motor4">
-      <hardwareInterface>hardware_interface/PositionJointInterface</hardwareInterface>
-      <mechanicalReduction>1</mechanicalReduction>
-    </actuator>
-  </transmission>
   <!-- Joint from upper_arm to lower_arm -->
   <!-- Note: 5-degree calibration offset applied to joint limits -->
@@ -416,39 +225,230 @@
     </actuator>
   </transmission>
-  <!-- Joint from shoulder to upper_arm -->
-  <joint name="shoulder_lift" type="revolute">
-    <origin xyz="-0.0303992 -0.0182778 -0.0542" rpy="${-pi/2} ${-pi/2} 0"/>
-    <parent link="shoulder_link"/>
-    <child link="upper_arm_link"/>
-    <axis xyz="0 0 1"/>
-    <limit effort="10" velocity="10" lower="-1.74533" upper="1.74533"/>
-  </joint>
-  <transmission name="shoulder_lift_trans">
-    <type>transmission_interface/SimpleTransmission</type>
-    <joint name="shoulder_lift">
-      <hardwareInterface>hardware_interface/PositionJointInterface</hardwareInterface>
-    </joint>
-    <actuator name="motor2">
-      <hardwareInterface>hardware_interface/PositionJointInterface</hardwareInterface>
-      <mechanicalReduction>1</mechanicalReduction>
-    </actuator>
-  </transmission>
-  <!-- Joint from base to shoulder -->
-  <joint name="shoulder_pan" type="revolute">
-    <origin xyz="0.0388353 0 0.0624" rpy="${pi} 0 ${-pi}"/>
-    <parent link="base_link"/>
-    <child link="shoulder_link"/>
-    <axis xyz="0 0 1"/>
-    <limit effort="10" velocity="10" lower="-1.91986" upper="1.91986"/>
-  </joint>
-  <transmission name="shoulder_pan_trans">
-    <type>transmission_interface/SimpleTransmission</type>
-    <joint name="shoulder_pan">
-      <hardwareInterface>hardware_interface/PositionJointInterface</hardwareInterface>
-    </joint>
-    <actuator name="motor1">
-      <hardwareInterface>hardware_interface/PositionJointInterface</hardwareInterface>
-      <mechanicalReduction>1</mechanicalReduction>
-    </actuator>
-  </transmission>
+  <!-- Link lower_arm -->
+  <link name="lower_arm_link">
+    <inertial>
+      <origin xyz="-0.0980701 0.00324376 0.0182831" rpy="0 0 0"/>
+      <mass value="0.104"/>
+      <inertia
+        ixx="2.87438e-05" ixy="7.41152e-06" ixz="1.26409e-06"
+        iyy="0.000159844" iyz="-4.90188e-08" izz="0.00014529"
+      />
+    </inertial>
+    <!-- Part under_arm_so101_v1 -->
+    <visual>
+      <origin xyz="-0.0648499 -0.032 0.0182" rpy="${pi} 0 0"/>
+      <geometry>
+        <mesh filename="package://so_arm_description/meshes/under_arm_so101_v1.stl"/>
+      </geometry>
+      <material name="3d_printed"/>
+    </visual>
+    <collision>
+      <origin xyz="-0.0648499 -0.032 0.0182" rpy="${pi} 0 0"/>
+      <geometry>
+        <mesh filename="package://so_arm_description/meshes/under_arm_so101_v1.stl"/>
+      </geometry>
+    </collision>
+    <!-- Part motor_holder_so101_wrist_v1 -->
+    <visual>
+      <origin xyz="-0.0648499 -0.032 0.018" rpy="${-pi} 0 0"/>
+      <geometry>
+        <mesh filename="package://so_arm_description/meshes/motor_holder_so101_wrist_v1.stl"/>
+      </geometry>
+      <material name="3d_printed"/>
+    </visual>
+    <collision>
+      <origin xyz="-0.0648499 -0.032 0.018" rpy="${-pi} 0 0"/>
+      <geometry>
+        <mesh filename="package://so_arm_description/meshes/motor_holder_so101_wrist_v1.stl"/>
+      </geometry>
+    </collision>
+    <!-- Part sts3215_03a_v1_4 -->
+    <visual>
+      <origin xyz="-0.1224 0.0052 0.0187" rpy="${-pi} 0 ${-pi}"/>
+      <geometry>
+        <mesh filename="package://so_arm_description/meshes/sts3215_03a_v1.stl"/>
+      </geometry>
+      <!-- <material name="sts3215"/> -->
+    </visual>
+    <collision>
+      <origin xyz="-0.1224 0.0052 0.0187" rpy="${-pi} 0 ${-pi}"/>
+      <geometry>
+        <mesh filename="package://so_arm_description/meshes/sts3215_03a_v1.stl"/>
+      </geometry>
+    </collision>
+  </link>
+  <!-- Joint from lower_arm to wrist -->
+  <joint name="wrist_flex" type="revolute">
+    <origin xyz="-0.1349 0.0052 0" rpy="0 0 ${-pi/2}"/>
+    <parent link="lower_arm_link"/>
+    <child link="wrist_link"/>
+    <axis xyz="0 0 1"/>
+    <limit effort="10" velocity="10" lower="-1.65806" upper="1.65806"/>
+  </joint>
+  <transmission name="wrist_flex_trans">
+    <type>transmission_interface/SimpleTransmission</type>
+    <joint name="wrist_flex">
+      <hardwareInterface>hardware_interface/PositionJointInterface</hardwareInterface>
+    </joint>
+    <actuator name="motor4">
+      <hardwareInterface>hardware_interface/PositionJointInterface</hardwareInterface>
+      <mechanicalReduction>1</mechanicalReduction>
+    </actuator>
+  </transmission>
+  <!-- Link wrist -->
+  <link name="wrist_link">
+    <inertial>
+      <origin xyz="-0.000103312 -0.0386143 0.0281156" rpy="0 0 0"/>
+      <mass value="0.079"/>
+      <inertia
+        ixx="3.68263e-05" ixy="1.7893e-08" ixz="-5.28128e-08"
+        iyy="2.5391e-05" iyz="3.6412e-06" izz="2.1e-05"
+      />
+    </inertial>
+    <!-- Part sts3215_03a_no_horn_v1 -->
+    <visual>
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
Commit message: Setting true velocity limit

File: so_arm_description/urdf/so_arm_101.urdf.xacro (robot description, xacro)
@@ -82,5 +82,5 @@
     <child link="shoulder_link"/>
     <axis xyz="0 0 1"/>
-    <limit effort="10" velocity="10" lower="-1.91986" upper="1.91986"/>
+    <limit effort="10" velocity="0.73" lower="-1.91986" upper="1.91986"/>
   </joint>
   <transmission name="shoulder_pan_trans">
@@ -154,5 +154,5 @@
     <child link="upper_arm_link"/>
     <axis xyz="0 0 1"/>
-    <limit effort="10" velocity="10" lower="-1.74533" upper="1.74533"/>
+    <limit effort="10" velocity="0.73" lower="-1.74533" upper="1.74533"/>
   </joint>
   <transmission name="shoulder_lift_trans">
@@ -213,5 +213,5 @@
     <child link="lower_arm_link"/>
     <axis xyz="0 0 1"/>
-    <limit effort="10" velocity="10" lower="-1.69" upper="1.58"/>
+    <limit effort="10" velocity="0.73" lower="-1.69" upper="1.58"/>
   </joint>
   <transmission name="elbow_flex_trans">
@@ -284,5 +284,5 @@
     <child link="wrist_link"/>
     <axis xyz="0 0 1"/>
-    <limit effort="10" velocity="10" lower="-1.65806" upper="1.65806"/>
+    <limit effort="10" velocity="0.73" lower="-1.65806" upper="1.65806"/>
   </joint>
   <transmission name="wrist_flex_trans">
@@ -342,5 +342,5 @@
     <child link="gripper_link"/>
     <axis xyz="0 0 1"/>
-    <limit effort="10" velocity="10" lower="-2.74385" upper="2.84121"/>
+    <limit effort="10" velocity="0.73" lower="-2.74385" upper="2.84121"/>
   </joint>
   <transmission name="wrist_roll_trans">
@@ -400,5 +400,5 @@
     <child link="moving_jaw_so101_v1_link"/>
     <axis xyz="0 0 1"/>
-    <limit effort="10" velocity="10" lower="-0.174533" upper="1.74533"/>
+    <limit effort="10" velocity="0.73" lower="-0.174533" upper="1.74533"/>
   </joint>
   <transmission name="gripper_trans">
