Commit message: Removing inertia from base_link

File: so_arm_description/urdf/so_arm_101.urdf.xacro (robot description, xacro)
@@ -11,4 +11,67 @@
   <!-- Link base -->
   <link name="base_link">
+    <!-- Part base_motor_holder_so101_v1 -->
+    <visual>
+      <origin xyz="-0.00636471 -9.94414e-05 -0.0024" rpy="${pi/2} 0 ${pi/2}"/>
+      <geometry>
+        <mesh filename="package://so_arm_description/meshes/base_motor_holder_so101_v1.stl"/>
+      </geometry>
+      <material name="3d_printed"/>
+    </visual>
+    <collision>
+      <origin xyz="-0.00636471 -9.94414e-05 -0.0024" rpy="${pi/2} 0 ${pi/2}"/>
+      <geometry>
+        <mesh filename="package://so_arm_description/meshes/base_motor_holder_so101_v1.stl"/>
+      </geometry>
+    </collision>
+    <!-- Part base_so101_v2 -->
+    <visual>
+      <origin xyz="-0.00636471 0 -0.0024" rpy="${pi/2} 0 ${pi/2}"/>
+      <geometry>
+        <mesh filename="package://so_arm_description/meshes/base_so101_v2.stl"/>
+      </geometry>
+      <material name="3d_printed"/>
+    </visual>
+    <collision>
+      <origin xyz="-0.00636471 0 -0.0024" rpy="${pi/2} 0 ${pi/2}"/>
+      <geometry>
+        <mesh filename="package://so_arm_description/meshes/base_so101_v2.stl"/>
+      </geometry>
+    </collision>
+    <!-- Part sts3215_03a_v1 -->
+    <visual>
+      <origin xyz="0.0263353 0 0.0437" rpy="0 0 0"/>
+      <geometry>
+        <mesh filename="package://so_arm_description/meshes/sts3215_03a_v1.stl"/>
+      </geometry>
+      <!-- <material name="sts3215"/> -->
+    </visual>
+    <collision>
+      <origin xyz="0.0263353 0 0.0437" rpy="0 0 0"/>
+      <geometry>
+        <mesh filename="package://so_arm_description/meshes/sts3215_03a_v1.stl"/>
+      </geometry>
+    </collision>
+    <!-- Part waveshare_mounting_plate_so101_v2 -->
+    <visual>
+      <origin xyz="-0.0309827 -0.000199441 0.0474" rpy="${pi/2} 0 ${pi/2}"/>
+      <geometry>
+        <mesh filename="package://so_arm_description/meshes/waveshare_mounting_plate_so101_v2.stl"/>
+      </geometry>
+      <material name="3d_printed"/>
+    </visual>
+    <collision>
+      <origin xyz="-0.0309827 -0.000199441 0.0474" rpy="${pi/2} 0 ${pi/2}"/>
+      <geometry>
+        <mesh filename="package://so_arm_description/meshes/waveshare_mounting_plate_so101_v2.stl"/>
+      </geometry>
+    </collision>
+  </link>
+  <joint name="base_link_inertia_joint" type="fixed">
+    <origin xyz="0 0 0" rpy="0 0 0"/>
+    <parent link="base_link"/>
+    <child link="base_link_inertia"/>
+  </joint>
+  <link name="base_link_inertia">
     <inertial>
       <origin xyz="0.0137179 -5.19711e-05 0.0334843" rpy="0 0 0"/>
@@ -19,60 +82,4 @@
       />
     </inertial>
-    <!-- Part base_motor_holder_so101_v1 -->
-    <visual>
-      <origin xyz="-0.00636471 -9.94414e-05 -0.0024" rpy="${pi/2} 0 ${pi/2}"/>
-      <geometry>
-        <mesh filename="package://so_arm_description/meshes/base_motor_holder_so101_v1.stl"/>
-      </geometry>
-      <material name="3d_printed"/>
-    </visual>
-    <collision>
-      <origin xyz="-0.00636471 -9.94414e-05 -0.0024" rpy="${pi/2} 0 ${pi/2}"/>
-      <geometry>
-        <mesh filename="package://so_arm_description/meshes/base_motor_holder_so101_v1.stl"/>
-      </geometry>
-    </collision>
-    <!-- Part base_so101_v2 -->
-    <visual>
-      <origin xyz="-0.00636471 0 -0.0024" rpy="${pi/2} 0 ${pi/2}"/>
-      <geometry>
-        <mesh filename="package://so_arm_description/meshes/base_so101_v2.stl"/>
-      </geometry>
-      <material name="3d_printed"/>
-    </visual>
-    <collision>
-      <origin xyz="-0.00636471 0 -0.0024" rpy="${pi/2} 0 ${pi/2}"/>
-      <geometry>
-        <mesh filename="package://so_arm_description/meshes/base_so101_v2.stl"/>
-      </geometry>
-    </collision>
-    <!-- Part sts3215_03a_v1 -->
-    <visual>
-      <origin xyz="0.0263353 0 0.0437" rpy="0 0 0"/>
-      <geometry>
-        <mesh filename="package://so_arm_description/meshes/sts3215_03a_v1.stl"/>
-      </geometry>
-      <!-- <material name="sts3215"/> -->
-    </visual>
-    <collision>
-      <origin xyz="0.0263353 0 0.0437" rpy="0 0 0"/>
-      <geometry>
-        <mesh filename="package://so_arm_description/meshes/sts3215_03a_v1.stl"/>
-      </geometry>
-    </collision>
-    <!-- Part waveshare_mounting_plate_so101_v2 -->
-    <visual>
-      <origin xyz="-0.0309827 -0.000199441 0.0474" rpy="${pi/2} 0 ${pi/2}"/>
-      <geometry>
-        <mesh filename="package://so_arm_description/meshes/waveshare_mounting_plate_so101_v2.stl"/>
-      </geometry>
-      <material name="3d_printed"/>
-    </visual>
-    <collision>
-      <origin xyz="-0.0309827 -0.000199441 0.0474" rpy="${pi/2} 0 ${pi/2}"/>
-      <geometry>
-        <mesh filename="package://so_arm_description/meshes/waveshare_mounting_plate_so101_v2.stl"/>
-      </geometry>
-    </collision>
   </link>
   <!-- Joint from base to shoulder -->
